File: lectrern hackpad PCB/lectrern hackpad.kicad_sch (KiCad schematic)
At the start: 18 parts, among them J1 oled connectors, SW1 SW_Push, SW2 SW_Push, SW3 SW_Push, SW4 SW_Push, SW5 SW_Push, SW6 SW_Push, U1 MOUDLE-SEEEDUINO-XIAO

Commit message: finish all the code firmware
Parts:
- D1, D2, D3, D4, D5, D6: footprint Diode_THT:D_5KPW_P7.62mm_Vertical_KathodeUp -> Diode_SMD:D_1206_3216Metric_Pad1.42x1.75mm_HandSolder
Changed lines of the file:
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@@
 			)
 		)
-		(property "Footprint" "Diode_THT:D_5KPW_P7.62mm_Vertical_KathodeUp"
+		(property "Footprint" "Diode_SMD:D_1206_3216Metric_Pad1.42x1.75mm_HandSolder"
 			(at 212.09 97.79 0)
 			(effects
@@
 			)
 		)
-		(property "Footprint" "Diode_THT:D_5KPW_P7.62mm_Vertical_KathodeUp"
+		(property "Footprint" "Diode_SMD:D_1206_3216Metric_Pad1.42x1.75mm_HandSolder"
 			(at 240.03 97.79 0)
 			(effects
@@
 			)
 		)
-		(property "Footprint" "Diode_THT:D_5KPW_P7.62mm_Vertical_KathodeUp"
+		(property "Footprint" "Diode_SMD:D_1206_3216Metric_Pad1.42x1.75mm_HandSolder"
 			(at 212.09 118.11 0)
 			(effects
@@
 			)
 		)
-		(property "Footprint" "Diode_THT:D_5KPW_P7.62mm_Vertical_KathodeUp"
+		(property "Footprint" "Diode_SMD:D_1206_3216Metric_Pad1.42x1.75mm_HandSolder"
 			(at 240.03 118.11 0)
 			(effects
@@
 			)
 		)
-		(property "Footprint" "Diode_THT:D_5KPW_P7.62mm_Vertical_KathodeUp"
+		(property "Footprint" "Diode_SMD:D_1206_3216Metric_Pad1.42x1.75mm_HandSolder"
 			(at 226.06 118.11 0)
 			(effects
@@
 			)
 		)
-		(property "Footprint" "Diode_THT:D_5KPW_P7.62mm_Vertical_KathodeUp"
+		(property "Footprint" "Diode_SMD:D_1206_3216Metric_Pad1.42x1.75mm_HandSolder"
 			(at 226.06 97.79 0)
 			(effects
